Commit message: fox name removed

File: ros_packages/src/rover/rover_description/urdf/base_rover_cart.gazebo.xacro (robot description, xacro)
@@ -1,6 +1,6 @@
 <?xml version="1.0"?>
-<robot name= "base_fox_cart" xmlns:xacro="http://ros.org/wiki/xacro" >
+<robot name= "base_rover_cart" xmlns:xacro="http://ros.org/wiki/xacro" >
 	<gazebo>
-		<plugin name= "base_fox_controller" filename="libgazebo_ros_diff_drive.so" >
+		<plugin name= "base_rover_controller" filename="libgazebo_ros_diff_drive.so" >
 			<commandTopic> cmd_vel </commandTopic>
 			<odometryTopic> odom </odometryTopic>

File: ros_packages/src/rover/rover_description/urdf/base_rover_cart.urdf.xacro (robot description, xacro)
@@ -1,14 +1,14 @@
 <?xml version="1.0" encoding="UTF-8"?>
-<robot name="base_fox_cart" xmlns:xacro="http://ros.org/wiki/xacro">
+<robot name="base_rover_cart" xmlns:xacro="http://ros.org/wiki/xacro">
 	<!--URDF uses SI Units: meters, radians and kilograms-->
 	<!-- common constants -->
-	<xacro:include filename="$(find fox_description)/urdf/common_properties.xacro"/>
-	<xacro:include filename="$(find fox_description)/urdf/wheel.urdf.xacro"/>
-	<xacro:include filename="$(find fox_description)/urdf/caster.urdf.xacro"/>
-	<xacro:include filename="$(find fox_description)/urdf/camera.urdf.xacro"/>
-	<xacro:include filename="$(find fox_description)/urdf/imu.urdf.xacro"/>
-	<xacro:include filename="$(find fox_description)/urdf/laser.urdf.xacro"/>
-	<xacro:include filename="$(find fox_description)/urdf/logo.urdf.xacro"/>
-	<!-- <xacro:include filename="$(find fox_description)/urdf/ar_tag.urdf.xacro"/> -->
+	<xacro:include filename="$(find rover_description)/urdf/common_properties.xacro"/>
+	<xacro:include filename="$(find rover_description)/urdf/wheel.urdf.xacro"/>
+	<xacro:include filename="$(find rover_description)/urdf/caster.urdf.xacro"/>
+	<xacro:include filename="$(find rover_description)/urdf/camera.urdf.xacro"/>
+	<xacro:include filename="$(find rover_description)/urdf/imu.urdf.xacro"/>
+	<xacro:include filename="$(find rover_description)/urdf/laser.urdf.xacro"/>
+	<xacro:include filename="$(find rover_description)/urdf/logo.urdf.xacro"/>
+	<!-- <xacro:include filename="$(find rover_description)/urdf/ar_tag.urdf.xacro"/> -->
 	<!-- Base
 	<link name="base_footprint"/>
@@ -22,5 +22,5 @@
             <origin xyz="0 0 0" rpy="0 0 0"/>
             <geometry>
-                <mesh filename="package://fox_description/meshes/fox_cart.dae"
+                <mesh filename="package://rover_description/meshes/rover_cart.dae"
 					scale="0.001 0.001 0.001"/>
 			</geometry>
@@ -57,4 +57,4 @@
 	</xacro:ar_tag> -->
 	<!-- Gazebo simulation plugins -->
-	<xacro:include filename="$(find fox_description)/urdf/base_fox_cart.gazebo.xacro"/>
+	<xacro:include filename="$(find rover_description)/urdf/base_rover_cart.gazebo.xacro"/>
 </robot>
