Commit message: modified:   README.md 	modified:   ros_packages/src/gazebo_environments/collapsed_house_description/launch/bringup_multi_uav_rover.launch 	modified:   ros_packages/src/gazebo_environments/collapsed_house_description/launch/start_gazebo_uav_rover_world.launch 	modified:   ros_packages/src/gazebo_environments/fire_station_description/launch/bringup_multi_uav_rover.launch 	modified:   ros_packages/src/gazebo_environments/fire_station_description/launch/start_gazebo_uav_rover_world.launch 	renamed:    ros_packages/src/rover/rover_description/urdf/base_fox_cart_verticaltag.urdf.xacro -> ros_packages/src/rover/rover_description/urdf/base_rover_cart_verticaltag.urdf.xacro 	modified:   ros_packages/src/rover/rover_description/urdf/camera.urdf.xacro 	modified:   ros_packages/src/rover/rover_description/urdf/laser.urdf.xacro 	modified:   ros_packages/src/rover/rover_description/urdf/wheel.urdf.xacro

File: ros_packages/src/rover/rover_description/urdf/base_rover_cart_verticaltag.urdf.xacro (robot description, xacro)
@@ -1,11 +1,11 @@
 <?xml version="1.0" encoding="UTF-8"?>
-<robot name="base_fox_cart_verticaltag" xmlns:xacro="http://ros.org/wiki/xacro">
+<robot name="base_rover_cart_verticaltag" xmlns:xacro="http://ros.org/wiki/xacro">
 	<!--URDF uses SI Units: meters, radians and kilograms-->
 	<!-- common constants -->
-	<!--xacro:include filename="$(find fox_description)/urdf/common_properties.xacro"/-->
+	<!--xacro:include filename="$(find rover_description)/urdf/common_properties.xacro"/-->
 	<!-- add wheel xacro platform include files -->
-	<xacro:include filename="$(find fox_description)/urdf/wheel.urdf.xacro"/>
-	<xacro:include filename="$(find fox_description)/urdf/caster.urdf.xacro"/>
-	<xacro:include filename="$(find fox_description)/urdf/ar_tag.urdf.xacro"/>
+	<xacro:include filename="$(find rover_description)/urdf/wheel.urdf.xacro"/>
+	<xacro:include filename="$(find rover_description)/urdf/caster.urdf.xacro"/>
+	<xacro:include filename="$(find rover_description)/urdf/ar_tag.urdf.xacro"/>
 	<!-- Base -->
 	<link name="base_footprint"/>
@@ -18,5 +18,5 @@
       		<origin xyz="0 0 0" rpy="0 0 0"/>
       		<geometry>
-        		<mesh 	filename="package://fox_description/meshes/base_cart.stl"
+        		<mesh 	filename="package://rover_description/meshes/base_cart.stl"
 						scale="0.001 0.001 0.001"/>
 			</geometry>
@@ -73,4 +73,4 @@
 	</xacro:ar_tag>
 	<!-- Gazebo simulation plugins -->
-	<xacro:include filename="$(find fox_description)/urdf/base_fox_cart.gazebo.xacro"/>
+	<xacro:include filename="$(find rover_description)/urdf/base_rover_cart.gazebo.xacro"/>
 </robot>

File: ros_packages/src/rover/rover_description/urdf/camera.urdf.xacro (robot description, xacro)
@@ -10,5 +10,5 @@
       <origin xyz="0 0 0" rpy="${pi/2} 0 ${pi/2}"/>
       <geometry>
-        <mesh filename="package://fox_description/meshes/astra.dae" scale="0.001 0.001 0.001" />
+        <mesh filename="package://rover_description/meshes/astra.dae" scale="0.001 0.001 0.001" />
       </geometry>
     </visual>

File: ros_packages/src/rover/rover_description/urdf/laser.urdf.xacro (robot description, xacro)
@@ -10,5 +10,5 @@
       <origin xyz="0 0 -0.15" rpy="0 0 0"/>
       <geometry>
-        <mesh filename="package://fox_description/meshes/lidar.dae" scale="0.001 0.001 0.001" />
+        <mesh filename="package://rover_description/meshes/lidar.dae" scale="0.001 0.001 0.001" />
       </geometry>
     </visual>

File: ros_packages/src/rover/rover_description/urdf/wheel.urdf.xacro (robot description, xacro)
@@ -14,5 +14,5 @@
 				<origin xyz="0 0 0" rpy="0 0 ${rz_}"/>
 				<geometry>
-					<mesh 	filename="package://fox_description/meshes/wheel_fox.dae"
+					<mesh 	filename="package://rover_description/meshes/wheel_rover.dae"
 							scale="0.001 0.001 0.001"/>
 				</geometry>
