Commit message: multi-robot namespacing rover

File: ros_packages/src/rover/rover_description/urdf/logo.urdf.xacro (robot description, xacro)
@@ -30,5 +30,5 @@
 			<kd value="0.2" />
 			<minDepth>0.001</minDepth>
-			<material>logo</material>
+			<material>logo_alm</material>
 		</gazebo>
 	</xacro:macro>
