Commit message: Fix rover_descriptions, added scripts for init and arming, Updated ReadMe.

File: ros_packages/src/rover/rover_description/urdf/ar_tag_multiple.urdf.xacro (robot description, xacro)
@@ -22,5 +22,5 @@
 		</link>
 		<joint name="ar_tag_${number_}_joint" type="fixed">
-			<parent link="base_cart_link"/>
+			<parent link="base_link"/>
 			<child link="ar_tag_${number_}"/>
 			<origin xyz= "${x_} ${y_} ${z_}" rpy="0.0 ${r_} 0.0"/>

File: ros_packages/src/rover/rover_description/urdf/base_rover_big_top.urdf.xacro (robot description, xacro)
@@ -1,22 +1,24 @@
 <?xml version="1.0" encoding="UTF-8"?>
-<robot name="base_rover" xmlns:xacro="http://ros.org/wiki/xacro">
+<robot name="base_rover_big_top" xmlns:xacro="http://ros.org/wiki/xacro">
 	<!--URDF uses SI Units: meters, radians and kilograms-->
 	<!-- common constants -->
-	<!--xacro:include filename="$(find rover_description)/urdf/common_properties.xacro"/-->
+	<xacro:include filename="$(find rover_description)/urdf/common_properties.xacro"/>
 	<!-- add wheel xacro platform include files -->
 	<xacro:include filename="$(find rover_description)/urdf/wheel.urdf.xacro"/>
 	<xacro:include filename="$(find rover_description)/urdf/caster.urdf.xacro"/>
-	<xacro:include filename="$(find rover_description)/urdf/ar_tag_multiple.urdf.xacro"/>
-	<!-- Base -->
+	<xacro:include filename="$(find rover_description)/urdf/logo_big.urdf.xacro"/>
+	<!-- <xacro:include filename="$(find rover_description)/urdf/ar_tag_multiple.urdf.xacro"/> -->
+	<!-- Base
 	<link name="base_footprint"/>
 	<joint name="base_joint" type="fixed">
- 		<parent link="base_footprint"/>
-	   	<child link="base_cart_link"/>
-	</joint>
-	<link name="base_cart_link">
+		<origin xyz="0 0 0.105" rpy="0 0 0"/>
+                <parent link="base_footprint"/>
+	        <child link="base_link"/>
+	</joint> -->
+	<link name="base_link">
     	<visual>
       		<origin xyz="0 0 0" rpy="0 0 0"/>
       		<geometry>
-        		<mesh 	filename="package://rover_description/meshes/base_cart.stl"
+        		<mesh filename="package://rover_description/meshes/rover_cart.dae"
 						scale="0.001 0.001 0.001"/>
 			</geometry>
@@ -24,41 +26,43 @@
     	</visual>
 		<collision>
-      		<origin xyz="-0.02 0 0.05" rpy="0 0 0"/>
-      		<geometry>
-        		<box size="0.44 0.28 0.10"/>
-      		</geometry>
+			<origin xyz="-0.225 0 0.05" rpy="0 0 0"/>
+			<geometry>
+				<box size="0.50 0.35 0.10"/>
+			</geometry>
 		</collision>
 		<inertial>
-      		<origin xyz="0 0 0" rpy="0 0 0"/>
-      		<mass value="5"/> <!-- in kg -->
+			<origin xyz="-0.225 0 0" rpy="0 0 0"/>
+			<mass value="20"/> <!-- in kg -->
 			<!-- M=20kg, x=0.5m, y=0.34m, z=0.1m-->
-      		<inertia ixx="0.2093333" ixy="0.0" ixz="0.0" iyy="0.4333333" iyz="0.0" izz="0.6093333"/>
-    	</inertial>
-  	</link>
+			<inertia ixx="0.2093333" ixy="0.0" ixz="0.0" iyy="0.4333333" iyz="0.0" izz="0.6093333"/>
+        </inertial>
+	</link>
 	<!-- front_wheel macros -->
-    <xacro:front_wheel alignment="left" x_="-0.229" y_="-0.12" z_="0.0005" r_="-1.5707" p_="0" j_="0" off_="-0.12" f_="0.01" s_="1.0"  >
+    <xacro:front_wheel alignment="left" x_="0" y_="0.25" z_="0" rx_="0" ry_="0" rz_="${pi}" off_="-0.12" f_="0.01" s_="1.0"  >
 	</xacro:front_wheel>
-    <xacro:front_wheel alignment="right" x_="-0.229" y_="0.12" z_="0.0005" r_="-1.5707" p_="0.0" j_="0.0" off_="0.12" f_="0.01" s_="1.0" >
+    <xacro:front_wheel alignment="right" x_="0" y_="-0.25" z_="0" rx_="0" ry_="0.0" rz_="0" off_="0.12" f_="0.01" s_="1.0" >
 	</xacro:front_wheel>
 	<!-- Caster macros -->
-    <!--<xacro:caster alignment="left" x_="0.188" y_="-0.2" z_="-0.047" >-->
-    <xacro:caster alignment="left" x_="0.188" y_="-0.2" z_="-0.047" >
+    <xacro:caster alignment="left" x_="-0.4" y_="-0.22" z_="-0.03" >
 	</xacro:caster>
-    <!--<xacro:caster alignment="right" x_="0.188" y_="0.2" z_="-0.047" >-->
-    <xacro:caster alignment="right" x_="0.188" y_="0.2" z_="-0.047" >
+    <xacro:caster alignment="right" x_="-0.4" y_="0.22" z_="-0.03" >
 	</xacro:caster>
+	<!-- logo macro -->
+	<xacro:logo_tag_big x_="-0.18" y_="0.0" z_="0.125" r_="0" p_="0" yaw_="0">
+	</xacro:logo_tag_big>
+	<!-- ar_tag macros -->
 	<!-- ar_tag macros top left-->
-    <xacro:ar_tag number_="5" x_="0.25" y_="0.25" z_="0.15" r_="0.0">
-	</xacro:ar_tag>
+    <!-- <xacro:ar_tag number_="5" x_="0.25" y_="0.25" z_="0.15" r_="0.0">
+	</xacro:ar_tag> -->
 	<!-- ar_tag macros bottom right-->
-    <xacro:ar_tag number_="13" x_="-0.25" y_="-0.25" z_="0.15" r_="0.0">
-	</xacro:ar_tag>
+    <!-- <xacro:ar_tag number_="13" x_="-0.25" y_="-0.25" z_="0.15" r_="0.0">
+	</xacro:ar_tag> -->
 	<!-- ar_tag macros top right-->
-    <xacro:ar_tag number_="1" x_="0.25" y_="-0.25" z_="0.15" r_="0.0">
-	</xacro:ar_tag>
+    <!-- <xacro:ar_tag number_="1" x_="0.25" y_="-0.25" z_="0.15" r_="0.0">
+	</xacro:ar_tag> -->
 	<!-- ar_tag macros bottom left-->
-    <xacro:ar_tag number_="2" x_="-0.25" y_="0.25" z_="0.15" r_="0.0">
-	</xacro:ar_tag>
+    <!-- <xacro:ar_tag number_="2" x_="-0.25" y_="0.25" z_="0.15" r_="0.0">
+	</xacro:ar_tag> -->
 	<!-- Gazebo simulation plugins -->
-	<xacro:include filename="$(find rover_description)/urdf/base_rover.gazebo.xacro"/>
+	<xacro:include filename="$(find rover_description)/urdf/base_rover_cart.gazebo.xacro"/>
 </robot>

Commit message: Added Ar tags to big top and modified launch files accordingly.

File: ros_packages/src/rover/rover_description/urdf/ar_tag_multiple.urdf.xacro (robot description, xacro)
@@ -6,5 +6,5 @@
 				<origin xyz="0 0 0" rpy="0 0 0"/>
 				<geometry>
-					<box size="0.5 0.5 0.03"/>
+					<box size="0.5 0.6 0.03"/>
 				</geometry>
 			</visual>
@@ -17,5 +17,5 @@
 				<origin xyz="0 0 0" rpy="0 0 0"/>
 				<geometry>
-					<box size="0.5 0.5 0.03"/>
+					<box size="0.5 0.75 0.03"/>
 				</geometry>
 			</collision>
@@ -29,4 +29,6 @@
 			<kp value="50000000.0" />
 			<kd value="0.2" />
+			<mu1 value="1.0"/>
+			<mu2 value="1.0"/>
 			<minDepth>0.001</minDepth>
                         <xacro:if value="${number_ == 5}">
@@ -36,5 +38,59 @@
                                 <material>ar_tag_13</material>
                         </xacro:if>
+                        <xacro:if value="${number_ == 1}">
+                                <material>logo_alm</material>
+                        </xacro:if>
+                        <xacro:if value="${number_ == 2}">
+                                <material>logo_alm</material>
+                        </xacro:if>
 		</gazebo>
+		<link name="ar_tag_${number_}_wall_1">
+			<visual>
+				<origin xyz="0 0 0" rpy="0 0 0"/>
+				<geometry>
+					<box size="0.5 0.01 0.025"/>
+				</geometry>
+			</visual>
+			<inertial>
+				<origin xyz="0 0 0"/>
+				<mass value="0.001" />
+				<inertia ixx="0.000001" ixy="0.0" ixz="0.0" iyy= "0.000001" iyz="0.0" izz="0.000001" />
+			</inertial>
+			<collision>
+				<origin xyz="0 0 0" rpy="0 0 0"/>
+				<geometry>
+					<box size="0.5 0.01 0.025"/>
+				</geometry>
+			</collision>
+		</link>
+		<joint name="ar_tag_${number_}_wall_joint_1" type="fixed">
+			<parent link="ar_tag_${number_}"/>
+			<child link="ar_tag_${number_}_wall_1"/>
+			<origin xyz="0 0.3 0.03" rpy="0 0 0"/>
+		</joint>
+		<link name="ar_tag_${number_}_wall_2">
+			<visual>
+				<origin xyz="0 0 0" rpy="0 0 0"/>
+				<geometry>
+					<box size="0.5 0.01 0.025"/>
+				</geometry>
+			</visual>
+			<inertial>
+				<origin xyz="0 0 0"/>
+				<mass value="0.001" />
+				<inertia ixx="0.000001" ixy="0.0" ixz="0.0" iyy= "0.000001" iyz="0.0" izz="0.000001" />
+			</inertial>
+			<collision>
+				<origin xyz="0 0 0" rpy="0 0 0"/>
+				<geometry>
+					<box size="0.5 0.01 0.025"/>
+				</geometry>
+			</collision>
+		</link>
+		<joint name="ar_tag_${number_}_wall_joint_2" type="fixed">
+			<parent link="ar_tag_${number_}"/>
+			<child link="ar_tag_${number_}_wall_2"/>
+			<origin xyz="0 -0.3 0.03" rpy="0 0 0"/>
+		</joint>
 	</xacro:macro>
 </robot>

File: ros_packages/src/rover/rover_description/urdf/base_rover_big_top.urdf.xacro (robot description, xacro)
@@ -4,9 +4,11 @@
 	<!-- common constants -->
 	<xacro:include filename="$(find rover_description)/urdf/common_properties.xacro"/>
-	<!-- add wheel xacro platform include files -->
 	<xacro:include filename="$(find rover_description)/urdf/wheel.urdf.xacro"/>
 	<xacro:include filename="$(find rover_description)/urdf/caster.urdf.xacro"/>
+	<xacro:include filename="$(find rover_description)/urdf/camera.urdf.xacro"/>
+	<xacro:include filename="$(find rover_description)/urdf/imu.urdf.xacro"/>
+	<xacro:include filename="$(find rover_description)/urdf/laser.urdf.xacro"/>
 	<xacro:include filename="$(find rover_description)/urdf/logo_big.urdf.xacro"/>
-	<!-- <xacro:include filename="$(find rover_description)/urdf/ar_tag_multiple.urdf.xacro"/> -->
+	<xacro:include filename="$(find rover_description)/urdf/ar_tag_multiple.urdf.xacro"/>
 	<!-- Base
 	<link name="base_footprint"/>
@@ -49,19 +51,19 @@
 	</xacro:caster>
 	<!-- logo macro -->
-	<xacro:logo_tag_big x_="-0.18" y_="0.0" z_="0.125" r_="0" p_="0" yaw_="0">
-	</xacro:logo_tag_big>
+	<!-- <xacro:logo_tag_big x_="-0.18" y_="0.0" z_="0.125" r_="0" p_="0" yaw_="0">
+	</xacro:logo_tag_big> -->
 	<!-- ar_tag macros -->
 	<!-- ar_tag macros top left-->
-    <!-- <xacro:ar_tag number_="5" x_="0.25" y_="0.25" z_="0.15" r_="0.0">
+    <!-- <xacro:ar_tag number_="2" x_="0.25" y_="0.25" z_="0.15" r_="0.0">
 	</xacro:ar_tag> -->
 	<!-- ar_tag macros bottom right-->
-    <!-- <xacro:ar_tag number_="13" x_="-0.25" y_="-0.25" z_="0.15" r_="0.0">
-	</xacro:ar_tag> -->
+    <xacro:ar_tag number_="13" x_="-0.36" y_="-0.3" z_="0.1" r_="0.0">
+	</xacro:ar_tag>
 	<!-- ar_tag macros top right-->
     <!-- <xacro:ar_tag number_="1" x_="0.25" y_="-0.25" z_="0.15" r_="0.0">
 	</xacro:ar_tag> -->
 	<!-- ar_tag macros bottom left-->
-    <!-- <xacro:ar_tag number_="2" x_="-0.25" y_="0.25" z_="0.15" r_="0.0">
-	</xacro:ar_tag> -->
+    <xacro:ar_tag number_="5" x_="-0.36" y_="0.3" z_="0.1" r_="0.0">
+	</xacro:ar_tag>
 	<!-- Gazebo simulation plugins -->
 	<xacro:include filename="$(find rover_description)/urdf/base_rover_cart.gazebo.xacro"/>

Commit message: Fixes for rover big top for two drones

File: ros_packages/src/rover/rover_description/urdf/ar_tag_multiple.urdf.xacro (robot description, xacro)
@@ -6,5 +6,5 @@
 				<origin xyz="0 0 0" rpy="0 0 0"/>
 				<geometry>
-					<box size="0.5 0.6 0.03"/>
+					<box size="0.5 0.8 0.03"/>
 				</geometry>
 			</visual>
@@ -17,5 +17,5 @@
 				<origin xyz="0 0 0" rpy="0 0 0"/>
 				<geometry>
-					<box size="0.5 0.75 0.03"/>
+					<box size="0.5 0.8 0.03"/>
 				</geometry>
 			</collision>
@@ -67,5 +67,5 @@
 			<parent link="ar_tag_${number_}"/>
 			<child link="ar_tag_${number_}_wall_1"/>
-			<origin xyz="0 0.3 0.03" rpy="0 0 0"/>
+			<origin xyz="0 0.4 0.03" rpy="0 0 0"/>
 		</joint>
 		<link name="ar_tag_${number_}_wall_2">
@@ -91,5 +91,5 @@
 			<parent link="ar_tag_${number_}"/>
 			<child link="ar_tag_${number_}_wall_2"/>
-			<origin xyz="0 -0.3 0.03" rpy="0 0 0"/>
+			<origin xyz="0 -0.4 0.03" rpy="0 0 0"/>
 		</joint>
 	</xacro:macro>

File: ros_packages/src/rover/rover_description/urdf/base_rover_big_top.urdf.xacro (robot description, xacro)
@@ -58,5 +58,5 @@
 	</xacro:ar_tag> -->
 	<!-- ar_tag macros bottom right-->
-    <xacro:ar_tag number_="13" x_="-0.36" y_="-0.3" z_="0.1" r_="0.0">
+    <xacro:ar_tag number_="13" x_="-0.36" y_="-0.4" z_="0.1" r_="0.0">
 	</xacro:ar_tag>
 	<!-- ar_tag macros top right-->
@@ -64,5 +64,5 @@
 	</xacro:ar_tag> -->
 	<!-- ar_tag macros bottom left-->
-    <xacro:ar_tag number_="5" x_="-0.36" y_="0.3" z_="0.1" r_="0.0">
+    <xacro:ar_tag number_="5" x_="-0.36" y_="0.4" z_="0.1" r_="0.0">
 	</xacro:ar_tag>
 	<!-- Gazebo simulation plugins -->
